Commit message: Update l_hand_y_joint

File: aero_description/typeJSK_hand/robots/aero.urdf (robot description, URDF)
Before this commit: robot AeroTypeFCESy, 69 links, 68 joints
Joints:
- joint l_hand_y_joint: origin xyz=-0.0 -0.02 -0.045 rpy=0 1.57079633 3.14159265 -> xyz=0.0 -0.02 -0.043 rpy=0 1.57079633 1.57079633
