Commit message: [aero_shop] Fix xacro:property tag

File: aero_shop/hand_yaw/urdf/hand_yaw.urdf.xacro (robot description, xacro)
@@ -6,5 +6,5 @@
        xmlns:xacro="http://ros.org/wiki/xacro">
   <xacro:include filename="$(find aero_description)/urdf/common.xacro" />
-  <property name="M_PI" value="3.1415926535897931" />
+  <xacro:property name="M_PI" value="3.1415926535897931" />
   <xacro:macro name="hand_yaw" params="prefix:=r reflect:=1 hand_link disable_mesh:=false">
   <!-- ============================   hand_yaw   ============================ -->
